Commit message: update

File: urdf/SO_7DOF_ARM100/urdf/SO_7DOF_ARM100.URDF (robot description, URDF)
Before this commit: robot SO_7DOF_ARM100_08h_HL_01d_URDF_01.SLDASM, 8 links, 7 joints
Links:
- link Base: geometry collision mesh filename=../meshes/Base.STL; visual mesh filename=../meshes/Base.STL
- link End_Servo: geometry collision mesh filename=../meshes/End_Servo.STL; visual mesh filename=../meshes/End_Servo.STL
- link Forearm: geometry collision mesh filename=../meshes/Forearm.STL; visual mesh filename=../meshes/Forearm.STL
- link Humeral_Elbow: geometry collision mesh filename=../meshes/Humeral_Elbow.STL; visual mesh filename=../meshes/Humeral_Elbow.STL
- link Shoulder_Pitch_Yaw: geometry collision mesh filename=../meshes/Shoulder_Pitch_Yaw.STL; visual mesh filename=../meshes/Shoulder_Pitch_Yaw.STL
- link Upper_Humeral: geometry collision mesh filename=../meshes/Upper_Humeral.STL; visual mesh filename=../meshes/Upper_Humeral.STL
- link Wrist_Roll_Yaw: geometry collision mesh filename=../meshes/Wrist_Roll_Yaw.STL; visual mesh filename=../meshes/Wrist_Roll_Yaw.STL
- link Wrist_Yaw_Pitch: geometry collision mesh filename=../meshes/Wrist_Yaw_Pitch.STL; visual mesh filename=../meshes/Wrist_Yaw_Pitch.STL
