Commit message: update

File: urdf/SO_5DOF_ARM100/urdf/SO_5DOF_ARM100.URDF (robot description, URDF)
Before this commit: robot SO_5DOF_ARM100_8j_URDF.SLDASM, 7 links, 6 joints
Joints:
- joint Elbow: limit (none) -> lower=-90 upper=90 effort=0 velocity=0
- joint Jaw: limit (none) -> lower=0 upper=90 effort=0 velocity=0
- joint Pitch: limit (none) -> lower=-90 upper=90 effort=0 velocity=0
- joint Rotation: limit (none) -> lower=-90 upper=90 effort=0 velocity=0
- joint Wrist_Pitch: limit (none) -> lower=-180 upper=0 effort=0 velocity=0
- joint Wrist_Roll: limit (none) -> lower=-90 upper=90 effort=0 velocity=0

Commit message: update

File: urdf/SO_5DOF_ARM100/urdf/SO_5DOF_ARM100.URDF (robot description, URDF)
Before this commit: robot SO_5DOF_ARM100, 7 links, 6 joints
Joints:
- joint Elbow: limit lower=-90 upper=90 effort=0 velocity=0 -> lower=-1.57 upper=1.57 effort=0 velocity=0; type continuous -> revolute
- joint Jaw: limit lower=0 upper=90 effort=0 velocity=0 -> lower=0 upper=1.57 effort=0 velocity=0; type continuous -> revolute
- joint Pitch: limit lower=-90 upper=90 effort=0 velocity=0 -> lower=-1.57 upper=1.57 effort=0 velocity=0; type continuous -> revolute
- joint Rotation: limit lower=-90 upper=90 effort=0 velocity=0 -> lower=-1.57 upper=1.57 effort=0 velocity=0; type continuous -> revolute
- joint Wrist_Pitch: limit lower=-180 upper=0 effort=0 velocity=0 -> lower=-3.14 upper=0 effort=0 velocity=0; type continuous -> revolute
- joint Wrist_Roll: limit lower=-90 upper=90 effort=0 velocity=0 -> lower=-1.57 upper=1.57 effort=0 velocity=0; type continuous -> revolute
